File: diplexer.kicad_pcb (KiCad board)
At the start: 2 copper layers, 157 x 72 mm, 41 parts, among them J1 Conn_Coaxial, J10 Conn_01x01_Pin, J11 Conn_01x01_Pin, J2 Conn_Coaxial, J3 Conn_Coaxial, J4 Conn_01x01_Pin, J5 Conn_01x01_Pin, J6 Conn_01x01_Pin, J7 Conn_01x01_Pin, J8 Conn_01x01_Pin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

Commit message: Add files via upload
Parts:
- moved J1 13.5 mm to (37.5, 65.6)
- moved L10 4.35 mm to (45.0, 83.5)
- moved J3 1.50 mm to (183.5, 80.3)
- moved J2 1.00 mm to (185.0, 49.4)
- moved C6 0.90 mm to (63.0, 84.9)
Connections:
- J1 pad 3: (no net) -> GND
Routing:
- net Net-(C16-Pad1): track 27.5 -> 22.9 mm
- net Net-(J1-In): track 45.5 -> 44.6 mm
Other:
- board text added: "4M"
- board text added: "HF+6M"
Changed lines of the file:
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@@
 	(footprint "sparkfun-electromech:L_Axial_L14.6-hand"
 		(layer "F.Cu")
-		(at 42.4 80)
+		(at 44.9875 83.5)
 		(descr "Inductor, Axial series, Axial, Horizontal, pin pitch=20.32mm, , length*diameter=16*9.5mm^2, Vishay, IM-10-37, http://www.vishay.com/docs/34030/im10.pdf")
 		(tags "Inductor Axial series Axial Horizontal pin pitch 20.32mm  length 16mm diameter 9.5mm Vishay IM-10-37")
@@
 	(footprint "sparkfun-electromech:1111"
 		(layer "F.Cu")
-		(at 62.1 84.89)
+		(at 63 84.89)
 		(property "Reference" "C6"
 			(at -1.75 0.65 90)
@@
 	(footprint "sparkfun-electromech:UHF slanted"
 		(layer "F.Cu")
-		(at 185 80.35 90)
+		(at 183.5 80.35 90)
 		(descr "UHF slanted")
 		(property "Reference" "J3"
@@
 	(footprint "sparkfun-electromech:N-conn slanted"
 		(layer "F.Cu")
-		(at 184 49.39 -90)
+		(at 185 49.39 -90)
 		(property "Reference" "J2"
-			(at -9.85 0 360)
+			(at -9.85 0 0)
 			(layer "F.SilkS")
 			(effects
@@
 	(footprint "sparkfun-electromech:UHF slanted"
 		(layer "F.Cu")
-		(at 37 52.11 -90)
+		(at 37.5 65.61 -90)
 		(descr "UHF slanted")
 		(property "Reference" "J1"
@@
 			(size 5 5)
 			(layers "F.Cu" "F.Paste" "F.Mask")
+			(net 3 "GND")
 		)
 	)
@@
 		)
 	)
+	(gr_text "HF+6M"
+		(at 165 74.5 0)
+		(layer "F.SilkS")
+		(effects
+			(font
+				(size 2 2)
+				(thickness 0.1)
+			)
+			(justify left bottom)
+		)
+	)
+	(gr_text "4M"
+		(at 168.5 44.5 0)
+		(layer "F.SilkS")
+		(effects
+			(font
+				(size 2 2)
+				(thickness 0.1)
+			)
+			(justify left bottom)
+		)
+	)
 	(dimension
 		(type aligned)
@@
 	)
 	(segment
-		(start 42.9967 79.4033)
+		(start 42.9967 65.5)
 		(end 42.9967 57.1958)
 		(width 2.39)
@@
 	)
 	(segment
-		(start 42.9967 53.4234)
-		(end 43.9133 54.34)
-		(width 2.39)
-		(layer "F.Cu")
-		(net 2)
-	)
-	(segment
 		(start 48.3 49.2)
 		(end 48.5 49)
@@
 	)
 	(segment
-		(start 42.9967 52.11)
-		(end 42.9967 53.4234)
-		(width 2.39)
-		(layer "F.Cu")
-		(net 2)
-	)
-	(segment
-		(start 41.8234 52.11)
-		(end 42.9967 52.11)
-		(width 2.39)
+		(start 42.8867 65.61)
+		(end 42.9967 65.5)
+		(width 2.7)
 		(layer "F.Cu")
 		(net 2)
 	)
 	(segment
-		(start 37 52.11)
-		(end 41.8234 52.11)
+		(start 44.9875 83.5)
+		(end 42.9967 81.5092)
 		(width 2.39)
 		(layer "F.Cu")
@@
 	)
 	(segment
-		(start 45.8525 54.34)
-		(end 43.9133 54.34)
+		(start 42.9967 81.5092)
+		(end 42.9967 65.5)
 		(width 2.39)
 		(layer "F.Cu")
@@
 	)
 	(segment
-		(start 42.4 80)
-		(end 42.9967 79.4033)
-		(width 2.39)
+		(start 37.5 65.61)
+		(end 42.8867 65.61)
+		(width 2.7)
 		(layer "F.Cu")
 		(net 2)
@@
 	)
 	(segment
-		(start 75.7667 44.5133)
-		(end 71.8 44.5133)
+		(start 76.84 43.44)
+		(end 75.7667 44.5133)
 		(width 2.39)
 		(layer "F.Cu")
@@
 	)
 	(segment
+		(start 71.8 44.5133)
+		(end 71.8 48.9)
+		(width 2.39)
+		(layer "F.Cu")
+		(net 5)
+	)
+	(segment
 		(start 71.8 52.9816)
 		(end 72.4792 53.6608)
@@
 	)
 	(segment
-		(start 71.8 48.9)
-		(end 71.8 44.5133)
-		(width 2.39)
-		(layer "F.Cu")
-		(net 5)
-	)
-	(segment
 		(start 95.6355 52.9816)
 		(end 95.3436 53.2735)
@@
 	)
 	(segment
-		(start 76.84 43.44)
-		(end 75.7667 44.5133)
-		(width 2.39)
-		(layer "F.Cu")
-		(net 5)
-	)
-	(segment
 		(start 96.3 52.9816)
 		(end 95.6355 52.9816)
@@
 	)
 	(segment
+		(start 75.7667 44.5133)
+		(end 71.8 44.5133)
+		(width 2.39)
+		(layer "F.Cu")
+		(net 5)
+	)
+	(segment
 		(start 72.8664 53.2736)
 		(end 95.3436 53.2736)
@@
 	(segment
 		(start 67.89 83.09)
-		(end 68.1 83.3)
+		(end 59.9975 83.09)
 		(width 2.39)
 		(layer "F.Cu")
@@
 	)
 	(segment
-		(start 63 83.09)
+		(start 68.1 83.3)
 		(end 67.89 83.09)
 		(width 2.39)
@@
 	)
 	(segment
-		(start 57 80)
-		(end 58.6133 81.6133)
-		(width 2.39)
-		(layer "F.Cu")
-		(net 8)
-	)
-	(segment
 		(start 71.8 83.3)
 		(end 77 88.5)
@@
 	)
 	(segment
-		(start 58.6133 81.6133)
-		(end 58.6133 83.09)
+		(start 59.9975 83.09)
+		(end 59.5875 83.5)
 		(width 2.39)
 		(layer "F.Cu")
@@
 		(width 2.39)
 		(layer "F.Cu")
-		(net 8)
-	)
-	(segment
-		(start 63 83.09)
-		(end 58.6133 83.09)
-		(width 2.39)
-		(layer "F.Cu")
