File: diplexer.kicad_pcb (KiCad board)
At the start: 2 copper layers, 157 x 72 mm, 41 parts, among them J1 Conn_Coaxial, J10 Conn_01x01_Pin, J11 Conn_01x01_Pin, J2 Conn_Coaxial, J3 Conn_Coaxial, J4 Conn_01x01_Pin, J5 Conn_01x01_Pin, J6 Conn_01x01_Pin, J7 Conn_01x01_Pin, J8 Conn_01x01_Pin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

Commit message: Add files via upload
Parts:
- moved C1 14.5 mm to (51.5, 67.9)
- moved C10 14.5 mm to (164.0, 97.0)
- moved C11 14.5 mm to (51.7, 62.6)
- moved C12 14.5 mm to (70.5, 62.5)
- moved C13 14.5 mm to (99.5, 62.5)
- moved C14 14.5 mm to (120.5, 62.5)
- moved C15 14.5 mm to (148.5, 63.5)
- moved C16 14.5 mm to (69.5, 100.5)
- moved C17 14.5 mm to (91.5, 100.5)
- moved C18 14.5 mm to (120.5, 98.5)
- moved C19 14.5 mm to (141.5, 98.5)
- moved C2 14.5 mm to (70.5, 67.9)
- moved C20 14.5 mm to (171.0, 98.0)
- moved C3 14.5 mm to (99.6, 67.9)
- moved C4 14.5 mm to (120.5, 67.9)
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Other:
- board size 157 x 72 mm -> 157 x 101 mm
- board text added: "TO RIG"
