File: diplexer.kicad_pcb (KiCad board)
At the start: 2 copper layers, 157 x 101 mm, 41 parts, among them J1 Conn_Coaxial, J10 Conn_01x01_Pin, J11 Conn_01x01_Pin, J2 Conn_Coaxial, J3 Conn_Coaxial, J4 Conn_01x01_Pin, J5 Conn_01x01_Pin, J6 Conn_01x01_Pin, J7 Conn_01x01_Pin, J8 Conn_01x01_Pin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

Commit message: Add files via upload
Parts:
- C1, C10, C11, C12, C13, C14, C15, C16, C17, C18, C19, C2, C20, C3, C4, C5, C6, C7, C8, C9: footprint sparkfun-electromech:1111 -> sparkfun-electromech:CAPC2927X178N
- moved C12 7.07 mm to (74.9, 68.0)
- moved C14 7.06 mm to (124.9, 68.0)
- moved C13 6.94 mm to (95.2, 67.9)
- moved C11 6.34 mm to (48.2, 67.9)
- moved C15 4.87 mm to (144.9, 66.8)
- moved C20 2.04 mm to (169.1, 97.3), turned to -90 degrees
- moved C19 1.64 mm to (140.3, 97.4), turned to -90 degrees
- moved C17 1.55 mm to (90.4, 99.4), turned to -90 degrees
- moved C6 1.38 mm to (64.7, 100.2), turned to 90 degrees
- moved C18 1.38 mm to (119.2, 98.0), turned to -90 degrees
- moved C5 1.38 mm to (149.5, 66.9)
- moved C1 0.88 mm to (52.4, 68.0)
- moved C8 0.52 mm to (114.4, 98.0), turned to 90 degrees
- moved C10 0.37 mm to (164.2, 97.3), turned to 90 degrees
- turned C16 to -90 degrees
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Routing:
- net Net-(C1-Pad2): track 26.0 -> 31.2 mm
- net Net-(J3-In): track 31.9 -> 27.9 mm
- net Net-(C13-Pad2): track 30.0 -> 33.9 mm
- net Net-(J2-In): track 32.1 -> 35.3 mm
- net Net-(J1-In): track 44.6 -> 47.2 mm
- net Net-(C17-Pad1): track 23.3 -> 25.2 mm
- net Net-(C14-Pad2): track 40.9 -> 42.5 mm
- net Net-(C12-Pad2): track 45.6 -> 44.3 mm
- net Net-(C19-Pad1): track 21.2 -> 22.1 mm
- net GND: vias 114 -> 110

Commit message: Add files via upload
Parts:
- moved C6 1.12 mm to (64.8, 101.3)
- moved C18 0.86 mm to (119.2, 98.9)
- moved C16 0.80 mm to (69.4, 101.3)
- moved C19 0.69 mm to (140.2, 98.1)
- moved C9 0.69 mm to (135.4, 98.1)
- moved C8 0.68 mm to (114.4, 98.7)
- moved C17 0.65 mm to (90.4, 100.1)
- moved C7 0.60 mm to (85.6, 100.0)
- moved C20 0.49 mm to (169.0, 97.8)
- moved C10 0.49 mm to (164.1, 97.8)
Routing:
- net Net-(C13-Pad2): track 33.9 -> 51.4 mm
- net Net-(C1-Pad2): track 31.2 -> 48.6 mm
- net Net-(C12-Pad2): track 44.3 -> 56.0 mm
- net Net-(J1-In): track 47.2 -> 57.7 mm
- net Net-(C14-Pad2): track 42.5 -> 52.4 mm
- net Net-(J2-In): track 35.3 -> 44.5 mm
- net Net-(C17-Pad1): track 25.2 -> 30.0 mm

Commit message: Add files via upload
Parts:
- moved L6 4.33 mm to (144.9, 98.8)
- moved C15 3.93 mm to (147.4, 69.8), turned to 0 degrees
- moved C3 3.67 mm to (97.0, 65.3), turned to 0 degrees
- moved C11 3.34 mm to (50.4, 70.3), turned to 0 degrees
- moved C4 3.15 mm to (122.7, 70.2), turned to 0 degrees
- moved C2 3.11 mm to (72.6, 70.2), turned to 0 degrees
- moved C12 3.11 mm to (72.7, 65.8), turned to 0 degrees
- moved C14 3.11 mm to (122.8, 65.8), turned to 0 degrees
- moved C10 2.75 mm to (165.0, 100.4)
- moved C20 2.75 mm to (169.9, 100.4)
- moved C19 2.71 mm to (140.3, 100.8)
- moved C9 2.71 mm to (135.5, 100.8)
- moved C1 2.60 mm to (50.5, 66.1), turned to 0 degrees
- moved C13 2.60 mm to (97.0, 69.8), turned to 0 degrees
- moved C5 2.58 mm to (147.5, 65.2), turned to 0 degrees
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Routing:
- net Net-(C1-Pad2): track 48.6 -> 28.5 mm
- net Net-(C13-Pad2): track 51.4 -> 34.7 mm
- net Net-(C12-Pad2): track 56.0 -> 39.4 mm
- net Net-(J1-In): track 57.7 -> 43.6 mm
- net Net-(C14-Pad2): track 52.4 -> 41.7 mm
- net Net-(J2-In): track 44.5 -> 36.2 mm
- net Net-(C17-Pad1): track 30.0 -> 23.6 mm
- net Net-(C18-Pad1): track 24.6 -> 22.2 mm
- net Net-(J3-In): track 27.9 -> 28.7 mm
- net GND: vias 110 -> 0

Commit message: Add files via upload
Parts:
- moved J2 0.90 mm to (186.4, 63.9)
Changed lines of the file:
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@@
 	(footprint "sparkfun-electromech:N-conn slanted"
 		(layer "F.Cu")
-		(at 185.5 63.89 -90)
+		(at 186.4 63.89 -90)
 		(property "Reference" "J2"
 			(at -9.85 0 0)

Commit message: Add files via upload
Added cutouts for connectors
Parts:
- removed J11, J8: Conn_01x01_Pin, MountingHole:MountingHole_3.2mm_M3_DIN965_Pad
- J1, J3: value Conn_Coaxial -> Conn_Coaxial_UHF; footprint sparkfun-electromech:UHF slanted -> sparkfun-electromech:UHF-slant-corr
- J2: value Conn_Coaxial -> Conn_Coaxial_N; footprint sparkfun-electromech:N-conn slanted -> sparkfun-electromech:Conn-N-slant-C
- moved J7 7.07 mm to (184.5, 40.5)
- moved J5 6.50 mm to (36.4, 41.0)
- moved J3 6.27 mm to (189.0, 98.6)
- moved J6 6.09 mm to (183.1, 117.1)
- moved J4 5.90 mm to (36.6, 117.4)
- moved J1 5.40 mm to (32.0, 80.2)
- moved J2 2.63 mm to (189.0, 63.9), turned to 90 degrees
Connections:
- J2 pad 3: GND -> (no net)
Routing:
- net Net-(J3-In): track 28.7 -> 21.2 mm
- net Net-(J1-In): track 43.6 -> 36.3 mm
- net GND: vias 0 -> 208
Other:
- board size 157 x 101 mm -> 157.1 x 101 mm
