File: diplexer.kicad_sch (KiCad schematic)
At the start: 41 parts, among them J1 Conn_Coaxial, J10 Conn_01x01_Pin, J11 Conn_01x01_Pin, J2 Conn_Coaxial, J3 Conn_Coaxial, J4 Conn_01x01_Pin, J5 Conn_01x01_Pin, J6 Conn_01x01_Pin, J7 Conn_01x01_Pin, J8 Conn_01x01_Pin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

Commit message: Add files via upload
Parts:
- C20: MPN (none) -> VJ1111D220JXRAJ
Changed lines of the file:
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@@
 			)
 		)
-		(property "MPN" ""
+		(property "MPN" "VJ1111D220JXRAJ "
 			(at 228.6 107.95 0)
 			(effects

Commit message: Add files via upload
Added cutouts for connectors
Parts:
- removed J11, J8: Conn_01x01_Pin, MountingHole:MountingHole_3.2mm_M3_DIN965_Pad, symbol Connector:Conn_01x01_Pin
- J1, J3: value Conn_Coaxial -> Conn_Coaxial_UHF; footprint sparkfun-electromech:UHF slanted -> sparkfun-electromech:UHF-slant-corr
- J2: value Conn_Coaxial -> Conn_Coaxial_N; footprint sparkfun-electromech:N-conn slanted -> sparkfun-electromech:Conn-N-slant-C
Changed lines of the file:
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@@
 	)
 	(junction
-		(at 85.09 165.1)
-		(diameter 0)
-		(color 0 0 0 0)
-	)
-	(junction
 		(at 58.42 146.05)
 		(diameter 0)
@@
 		(color 0 0 0 0)
 	)
-	(junction
-		(at 85.09 147.32)
-		(diameter 0)
-		(color 0 0 0 0)
-	)
 	(wire
 		(pts
@@
 	(wire
 		(pts
-			(xy 85.09 165.1) (xy 85.09 166.37)
+			(xy 85.09 157.48) (xy 85.09 166.37)
 		)
 		(stroke
@@
 	(wire
 		(pts
-			(xy 85.09 157.48) (xy 85.09 165.1)
-		)
-		(stroke
-			(width 0)
-			(type default)
-		)
-	)
-	(wire
-		(pts
 			(xy 144.78 104.14) (xy 156.21 104.14)
 		)
@@
 	(wire
 		(pts
-			(xy 85.09 138.43) (xy 85.09 147.32)
-		)
-		(stroke
-			(width 0)
-			(type default)
-		)
-	)
-	(wire
-		(pts
 			(xy 156.21 104.14) (xy 168.91 104.14)
 		)
@@
 	)
 	(symbol
-		(lib_id "Connector:Conn_01x01_Pin")
-		(at 80.01 138.43 0)
-		(unit 1)
-		(exclude_from_sim no)
-		(in_bom yes)
-		(on_board yes)
-		(dnp no)
-		(fields_autoplaced yes)
-		(property "Reference" "J8"
-			(at 80.645 133.35 0)
-			(effects
-				(font
-					(size 1.27 1.27)
-				)
-			)
-		)
-		(property "Value" "Conn_01x01_Pin"
-			(at 80.645 135.89 0)
-			(effects
-				(font
-					(size 1.27 1.27)
-				)
-			)
-		)
-		(property "Footprint" "MountingHole:MountingHole_3.2mm_M3_DIN965_Pad"
-			(at 80.01 138.43 0)
-			(effects
-				(font
-					(size 1.27 1.27)
-				)
-				(hide yes)
-			)
-		)
-		(property "Datasheet" "~"
-			(at 80.01 138.43 0)
-			(effects
-				(font
-					(size 1.27 1.27)
-				)
-				(hide yes)
-			)
-		)
-		(property "Description" "Generic connector, single row, 01x01, script generated"
-			(at 80.01 138.43 0)
-			(effects
-				(font
-					(size 1.27 1.27)
-				)
-				(hide yes)
-			)
-		)
-		(pin "1"
-		)
-		(instances
-			(project "diplexer"
-				(path "/e3e6d633-5780-4393-92a9-d0fa1a8bbdfb"
-					(reference "J8")
-					(unit 1)
-				)
-			)
-		)
-	)
-	(symbol
-		(lib_id "Connector:Conn_01x01_Pin")
-		(at 80.01 165.1 0)
-		(unit 1)
-		(exclude_from_sim no)
-		(in_bom yes)
-		(on_board yes)
-		(dnp no)
-		(fields_autoplaced yes)
-		(property "Reference" "J11"
-			(at 80.645 160.02 0)
-			(effects
-				(font
-					(size 1.27 1.27)
-				)
-			)
-		)
-		(property "Value" "Conn_01x01_Pin"
-			(at 80.645 162.56 0)
-			(effects
-				(font
-					(size 1.27 1.27)
-				)
-			)
-		)
-		(property "Footprint" "MountingHole:MountingHole_3.2mm_M3_DIN965_Pad"
-			(at 80.01 165.1 0)
-			(effects
-				(font
-					(size 1.27 1.27)
-				)
-				(hide yes)
-			)
-		)
-		(property "Datasheet" "~"
-			(at 80.01 165.1 0)
-			(effects
-				(font
-					(size 1.27 1.27)
-				)
-				(hide yes)
-			)
-		)
-		(property "Description" "Generic connector, single row, 01x01, script generated"
-			(at 80.01 165.1 0)
-			(effects
-				(font
-					(size 1.27 1.27)
-				)
-				(hide yes)
-			)
-		)
-		(pin "1"
-		)
-		(instances
-			(project "diplexer"
-				(path "/e3e6d633-5780-4393-92a9-d0fa1a8bbdfb"
-					(reference "J11")
-					(unit 1)
-				)
-			)
-		)
-	)
-	(symbol
 		(lib_id "power:GND")
 		(at 228.6 111.76 0)
@@
 			)
 		)
-		(property "Value" "Conn_Coaxial"
+		(property "Value" "Conn_Coaxial_UHF"
 			(at 248.92 105.7031 0)
 			(effects
@@
 			)
 		)
-		(property "Footprint" "sparkfun-electromech:UHF slanted"
+		(property "Footprint" "sparkfun-electromech:UHF-slant-corr"
 			(at 245.11 104.14 0)
 			(effects
@@
 			)
 		)
-		(property "Value" "Conn_Coaxial"
-			(at 29.21 54.9031 0)
+		(property "Value" "Conn_Coaxial_UHF"
+			(at 29.972 54.864 0)
 			(effects
 				(font
@@
 			)
 		)
-		(property "Footprint" "sparkfun-electromech:UHF slanted"
+		(property "Footprint" "sparkfun-electromech:UHF-slant-corr"
 			(at 33.02 53.34 0)
 			(effects
@@
 		(fields_autoplaced yes)
 		(property "Reference" "J2"
-			(at 213.36 52.3631 0)
+			(at 212.09 52.3631 0)
 			(effects
 				(font
@@
 			)
 		)
-		(property "Value" "Conn_Coaxial"
-			(at 213.36 54.9031 0)
+		(property "Value" "Conn_Coaxial_N"
+			(at 212.09 54.9031 0)
 			(effects
 				(font
@@
 			)
 		)
-		(property "Footprint" "sparkfun-electromech:N-conn slanted"
+		(property "Footprint" "sparkfun-electromech:Conn-N-slant-C"
 			(at 209.296 44.45 0)
 			(effects
